Commit message: gazebo urdf files added

File: src/my_first_ros_package/robot_urdf/my_robot.urdf (robot description, URDF)
Before this commit: robot robot_1, 6 links, 5 joints
Links:
- link base_link: mass None -> 10.216; geometry collision cylinder length=0.03 radius=0.2; visual cylinder length=0.03 radius=0.2
- link castor_1: mass None -> 1.419; geometry collision sphere radius=0.05; visual sphere radius=0.05
- link castor_2: mass None -> 1.419; geometry collision sphere radius=0.05; visual sphere radius=0.05
- link left_wheel: mass None -> 0.8514; geometry collision cylinder length=0.04 radius=0.05; visual cylinder length=0.04 radius=0.05
- link right_wheel: mass None -> 0.8514; geometry collision cylinder length=0.04 radius=0.05; visual cylinder length=0.04 radius=0.05
Joints:
- joint support_back: origin xyz=-0.2 0.0 -0.06 rpy=0 0 0 -> xyz=-0.2 0.0 -0.065 rpy=0 0 0
- joint support_front: origin xyz=0.2 0.0 -0.06 rpy=0 0 0 -> xyz=0.2 0.0 -0.065 rpy=0 0 0

Commit message: added castor_1 and castor_2 gazebo blocks + added colours to the parts

File: src/my_first_ros_package/robot_urdf/my_robot.urdf (robot description, URDF)
Before this commit: robot robot_1, 6 links, 5 joints
Joints:
- joint right_wheel_joint: origin xyz=0 -0.22 -0.065 rpy=1.570796 0 0 -> xyz=0 -0.22 -0.065 rpy=-1.570796 0 0
